Commit message: Modified visual mesh.

File: urdf/oslsim.urdf (robot description, URDF)
Before this commit: robot oslsim, 8 links, 7 joints
Links:
- link footL: geometry collision mesh filename=package://oslsim/meshes/footLCollider.STL; visual mesh filename=package://oslsim/meshes/footL.dae
- link footR: geometry collision mesh filename=package://oslsim/meshes/footRCollider.STL; visual mesh filename=package://oslsim/meshes/footR.dae
- link pylonL: geometry collision mesh filename=package://oslsim/meshes/pylonLCollider.STL; visual mesh filename=package://oslsim/meshes/pylonL.dae
- link pylonR: geometry collision mesh filename=package://oslsim/meshes/pylonRCollider.STL; visual mesh filename=package://oslsim/meshes/pylonR.dae
- link thighL: geometry collision mesh filename=package://oslsim/meshes/thighLCollider.STL; visual mesh filename=package://oslsim/meshes/thighL.dae
- link thighR: geometry collision mesh filename=package://oslsim/meshes/thighRCollider.STL; visual mesh filename=package://oslsim/meshes/thighR.dae

Commit message: Minor bug fixes.

File: urdf/oslsim.urdf (robot description, URDF)
Before this commit: robot oslsim, 8 links, 7 joints
Joints:
- joint ankleL: limit lower=-1.57 upper=1.57 effort=1000.0 velocity=50 -> lower=-1.57 upper=1.57 effort=10.0 velocity=1000
- joint ankleR: limit lower=-1.57 upper=1.57 effort=1000.0 velocity=50 -> lower=-1.57 upper=1.57 effort=10.0 velocity=1000
- joint hipL: limit lower=-1.57 upper=1.57 effort=1000.0 velocity=50 -> lower=-1.57 upper=1.57 effort=10.0 velocity=1000
- joint hipR: limit lower=-1.57 upper=1.57 effort=1000.0 velocity=50 -> lower=-1.57 upper=1.57 effort=10.0 velocity=1000
- joint kneeL: limit lower=-1.57 upper=1.57 effort=1000.0 velocity=50 -> lower=-1.57 upper=1.57 effort=10.0 velocity=1000
- joint kneeR: limit lower=-1.57 upper=1.57 effort=1000.0 velocity=50 -> lower=-1.57 upper=1.57 effort=10.0 velocity=1000

Commit message: Fixed major bugs.

File: urdf/oslsim.urdf (robot description, URDF)
Before this commit: robot oslsim, 8 links, 7 joints
Links:
- removed link root
- added link entity, mass 0.01
- added link slider, mass 0.0001; collision box size=0.25 0.25 0.01
- added link world
- link footL: geometry collision box size=0.05 0.05 0.22; visual mesh filename=package://oslsim/meshes/footL.dae
- link footR: geometry collision box size=0.05 0.05 0.22; visual mesh filename=package://oslsim/meshes/footR.dae
- link pylonL: geometry collision box size=0.1 0.35 0.1; visual mesh filename=package://oslsim/meshes/pylonL.dae
- link pylonR: geometry collision box size=0.1 0.35 0.1; visual mesh filename=package://oslsim/meshes/pylonR.dae
- link thighL: geometry collision box size=0.15 0.3 0.15; visual mesh filename=package://oslsim/meshes/thighL.dae
- link thighR: geometry collision box size=0.15 0.3 0.15; visual mesh filename=package://oslsim/meshes/thighR.dae
Joints:
- added joint entity_joint: type fixed, parent slider, child entity, origin xyz=0 0 -0.045 rpy=0 0 0
- added joint slider_joint: type prismatic, parent world, child slider, origin xyz=0 0 0 rpy=0.0 0.0 0.0, axis 1 0 0, limit lower=-10.0 upper=100.0 effort=100 velocity=1
- joint root_joint: parent root -> entity

Commit message: Fixed OSL props.

File: urdf/oslsim.urdf (robot description, URDF)
Before this commit: robot oslsim, 10 links, 9 joints
Links:
- link footL: geometry collision box size=0.0675 0.025 0.22; visual mesh filename=package://oslsim/meshes/footL.dae
- link footR: geometry collision box size=0.0675 0.025 0.22; visual mesh filename=package://oslsim/meshes/footR.dae
- link slider: mass 0.0001 -> 1.0
Joints:
- joint ankleL: limit lower=-1.57 upper=1.57 effort=10.0 velocity=1000 -> lower=-1.57 upper=1.57 effort=1.0 velocity=100
- joint ankleR: limit lower=-1.57 upper=1.57 effort=10.0 velocity=1000 -> lower=-1.57 upper=1.57 effort=1.0 velocity=100
- joint entity_joint: origin xyz=0 0 -0.045 rpy=0 0 0 -> xyz=0 0 -0.05 rpy=0 0 0
- joint hipL: limit lower=-1.57 upper=1.57 effort=10.0 velocity=1000 -> lower=-1.57 upper=1.57 effort=1.0 velocity=100
- joint hipR: limit lower=-1.57 upper=1.57 effort=10.0 velocity=1000 -> lower=-1.57 upper=1.57 effort=1.0 velocity=100
- joint kneeL: limit lower=-1.57 upper=1.57 effort=10.0 velocity=1000 -> lower=-1.57 upper=1.57 effort=1.0 velocity=100
- joint kneeR: limit lower=-1.57 upper=1.57 effort=10.0 velocity=1000 -> lower=-1.57 upper=1.57 effort=1.0 velocity=100
- joint slider_joint: limit lower=-10.0 upper=100.0 effort=100 velocity=1 -> lower=-10.0 upper=100.0 effort=100 velocity=10

Commit message: Added sensors.

File: urdf/oslsim.urdf (robot description, URDF)
Before this commit: robot oslsim, 10 links, 9 joints
Links:
- added link footL_loadcell_link, mass 0.0001; collision sphere radius=0.020; visual sphere radius=0.020
- added link footR_loadcell_link, mass 0.0001; collision sphere radius=0.020; visual sphere radius=0.020
Joints:
- added joint footL_loadcell_link_joint: type fixed, parent footL, child footL_loadcell_link, origin xyz=0.03 -0.07 0 rpy=0 0 0
- added joint footR_loadcell_link_joint: type fixed, parent footR, child footR_loadcell_link, origin xyz=0.03 0.07 0 rpy=0 0 0

Commit message: Bug Fix #01

File: urdf/oslsim.urdf (robot description, URDF)
Before this commit: robot oslsim, 12 links, 11 joints
Links:
- link body: mass 0.001 -> 0.1
- link entity: mass 0.01 -> 0.001
- link footL: mass 0.19826 -> 0.79826; geometry collision box size=0.0675 0.025 0.2; visual mesh filename=package://oslsim/meshes/footL.dae
- link footL_loadcell_link: geometry collision sphere radius=0.020
- link footR: mass 0.19826 -> 0.79826; geometry collision box size=0.0675 0.025 0.2; visual mesh filename=package://oslsim/meshes/footR.dae
- link footR_loadcell_link: geometry collision sphere radius=0.020
- link slider: mass 1.0 -> 0.001
Joints:
- joint footL_loadcell_link_joint: origin xyz=0.03 -0.07 0 rpy=0 0 0 -> xyz=0.03 -0.06 0 rpy=0 0 0
- joint footR_loadcell_link_joint: origin xyz=0.03 0.07 0 rpy=0 0 0 -> xyz=0.03 0.06 0 rpy=0 0 0

Commit message: Modified joint dynamics.

File: urdf/oslsim.urdf (robot description, URDF)
Before this commit: robot oslsim, 12 links, 11 joints
Links:
- link entity: mass 0.001 -> 0.1
- link footL: mass 0.79826 -> 0.001
- link footL_loadcell_link: mass 0.0001 -> 0.00001
- link footR: mass 0.79826 -> 0.001
- link footR_loadcell_link: mass 0.0001 -> 0.00001
- link pylonL: mass 0.93649 -> 0.093649
- link pylonR: mass 0.9365 -> 0.09365
- link thighL: mass 5.5797 -> 0.55797
- link thighR: mass 5.5993 -> 0.55993
Joints:
- joint slider_joint: limit lower=-10.0 upper=100.0 effort=100 velocity=10 -> lower=-10.0 upper=100.0 effort=1 velocity=10

Commit message: Updated loadcell position.

File: urdf/oslsim.urdf (robot description, URDF)
Before this commit: robot oslsim, 12 links, 11 joints
Joints:
- joint footL_loadcell_link_joint: origin xyz=0.03 -0.06 0 rpy=0 0 0 -> xyz=0.03 -0.065 0 rpy=0 0 0
- joint footR_loadcell_link_joint: origin xyz=0.03 0.06 0 rpy=0 0 0 -> xyz=0.03 0.065 0 rpy=0 0 0

Commit message: Updated URDF.

File: urdf/oslsim.urdf (robot description, URDF)
Before this commit: robot oslsim, 12 links, 11 joints
Links:
- removed link footL_loadcell_link
- added link footL_heel, mass 0.00001; collision sphere radius=0.020
- link footL: geometry collision box size=0.0675 0.025 0.2; visual mesh filename=package://oslsim/meshes/foot.dae
- link pylonL: geometry collision box size=0.1 0.35 0.1; visual mesh filename=package://oslsim/meshes/pylon.dae
- link thighL: geometry collision box size=0.15 0.3 0.15; visual mesh filename=package://oslsim/meshes/thigh.dae
- link thighR: geometry collision box size=0.15 0.3 0.15; visual mesh filename=package://oslsim/meshes/socket.dae
Joints:
- removed joint footL_loadcell_link_joint
- added joint footL_heel_joint: type fixed, parent footL, child footL_heel, origin xyz=0.03 -0.065 0 rpy=0 0 0

Commit message: Fixed ground friction.

File: urdf/oslsim.urdf (robot description, URDF)
Before this commit: robot oslsim, 12 links, 11 joints
Joints:
- joint hipL: origin xyz=0 0 0 rpy=0 0 0 -> xyz=-0.015 0 0 rpy=0 0 0
- joint slider_joint: limit lower=-10.0 upper=100.0 effort=1 velocity=10 -> lower=-10.0 upper=100.0 effort=1 velocity=1

Commit message: Bug Fix #02

File: urdf/oslsim.urdf (robot description, URDF)
Before this commit: robot oslsim, 12 links, 11 joints
Links:
- removed link footL
- removed link footL_heel
- removed link footR
- removed link footR_loadcell_link
- removed link pylonL
- removed link pylonR
- removed link thighL
- removed link thighR
- added link foot, mass 0.001; collision box size=0.0675 0.025 0.2; visual mesh filename=package://oslsim/meshes/foot.dae
- added link foot_heel, mass 0.00001; collision sphere radius=0.020
- added link osl_foot, mass 0.001; collision box size=0.0675 0.025 0.2; visual mesh filename=package://oslsim/meshes/osl_foot.dae
- added link osl_foot_loadcell_link, mass 0.00001; collision sphere radius=0.020
- added link osl_shank, mass 0.09365; collision box size=0.1 0.35 0.1; visual mesh filename=package://oslsim/meshes/pylonR.dae
- added link shin, mass 0.093649; collision box size=0.1 0.35 0.1; visual mesh filename=package://oslsim/meshes/shin.dae
- added link socket, mass 0.55993; collision box size=0.15 0.3 0.15; visual mesh filename=package://oslsim/meshes/socket.dae
- added link thigh, mass 0.55797; collision box size=0.15 0.3 0.15; visual mesh filename=package://oslsim/meshes/thigh.dae
Joints:
- removed joint ankleL
- removed joint ankleR
- removed joint footL_heel_joint
- removed joint footR_loadcell_link_joint
- removed joint hipL
- removed joint hipR
- removed joint kneeL
- removed joint kneeR
- added joint ankle: type revolute, parent shin, child foot, origin xyz=-0.00077967 -0.3134 -0.026811 rpy=0 1.5708 0, axis 1 0 0, limit lower=-1.57 upper=1.57 effort=1.0 velocity=100
- added joint foot_heel_joint: type fixed, parent foot, child foot_heel, origin xyz=0.03 -0.065 0 rpy=0 0 0
- added joint hip: type revolute, parent body, child thigh, origin xyz=-0.03 0 0 rpy=0 0 0, axis -0.03 1 0, limit lower=-1.57 upper=1.57 effort=1.0 velocity=100
- added joint knee: type revolute, parent thigh, child shin, origin xyz=-0.0073766 0.057865 -0.4427 rpy=1.5708 0 0, axis 0 0 1, limit lower=-1.57 upper=1.57 effort=1.0 velocity=100
- added joint osl_ankle: type revolute, parent osl_shank, child osl_foot, origin xyz=-0.00077967 -0.3134 0.026811 rpy=-3.1416 -1.5708 0, axis 1 0 0, limit lower=-1.57 upper=1.57 effort=1.0 velocity=100
- added joint osl_foot_loadcell_link_joint: type fixed, parent osl_foot, child osl_foot_loadcell_link, origin xyz=0.03 0.065 0 rpy=0 0 0
- added joint osl_hip: type revolute, parent body, child socket, origin xyz=0 0 0 rpy=0 0 0, axis 0 1 0, limit lower=-1.57 upper=1.57 effort=1.0 velocity=100
- added joint osl_knee: type revolute, parent socket, child osl_shank, origin xyz=-0.0073766 -0.062441 -0.4427 rpy=1.5708 0 0, axis 0 0 1, limit lower=-1.57 upper=1.57 effort=1.0 velocity=100

Commit message: Removed pylon.

File: urdf/oslsim.urdf (robot description, URDF)
Before this commit: robot oslsim, 12 links, 11 joints
Links:
- link osl_shank: geometry collision box size=0.1 0.35 0.1; visual mesh filename=package://oslsim/meshes/osl_shank.dae

Commit message: Added controller node.

File: urdf/oslsim.urdf (robot description, URDF)
Before this commit: robot oslsim, 12 links, 11 joints
Joints:
- joint hip: origin xyz=-0.03 0 0 rpy=0 0 0 -> xyz=-0.03 -0.015 0 rpy=0 0 0
- joint osl_hip: origin xyz=0 0 0 rpy=0 0 0 -> xyz=0 0.015 0 rpy=0 0 0
