Commit message: Added motors.

File: urdf/oslsim.xacro (robot description, xacro)
@@ -1,4 +1,5 @@
 <?xml version="1.0" encoding="utf-8"?>
-<robot name="oslsim">
+<robot name="oslsim" xmlns:xacro="http://www.ros.org/wiki/xacro">
+  <xacro:include filename="$(find gazebo_ros_motors)/xacro/dc_motor.xacro"/>
   <gazebo>
     <plugin name="gazebo_ros_control" filename="libgazebo_ros_control.so">
@@ -6,4 +7,20 @@
     </plugin>
   </gazebo>
+  <xacro:dc_motor motor_name="osl_ankle" parent_link="osl_shank" child_link="osl_foot">
+    <xacro:property name="params_yaml" value="$(find oslsim)/config/osl_ankle.yaml"/>
+    <origin
+      xyz="-0.00077967 -0.3134 0.026811"
+      rpy="-3.1416 -1.5708 0" />
+    <axis
+      xyz="1 0 0" />
+  </xacro:dc_motor>
+  <xacro:dc_motor motor_name="osl_knee" parent_link="socket" child_link="osl_shank">
+    <xacro:property name="params_yaml" value="$(find oslsim)/config/osl_knee.yaml"/>
+    <origin
+      xyz="-0.0073766 -0.062441 -0.4427"
+      rpy="1.5708 0 0" />
+    <axis
+      xyz="0 0 1" />
+  </xacro:dc_motor>
   <gazebo>
       <plugin name="p3d_base_controller" filename="libgazebo_ros_p3d.so">
@@ -347,5 +364,5 @@
     </actuator>
   </transmission>
-  <joint name="osl_knee" type="revolute">
+  <!-- <joint name="osl_knee" type="revolute">
     <origin
       xyz="-0.0073766 -0.062441 -0.4427"
@@ -369,5 +386,5 @@
       <mechanicalReduction>1</mechanicalReduction>
     </actuator>
-  </transmission>
+  </transmission> -->
   <link name="foot">
     <inertial>
@@ -540,5 +557,5 @@
     </actuator>
   </transmission>
-  <joint name="osl_ankle"
+  <!-- <joint name="osl_ankle"
     type="revolute">
     <origin
@@ -563,5 +580,5 @@
       <mechanicalReduction>1</mechanicalReduction>
     </actuator>
-  </transmission>
+  </transmission> -->
   <link name="foot_heel">
     <inertial>

Commit message: Fixed ankle motor.

File: urdf/oslsim.xacro (robot description, xacro)
@@ -11,7 +11,5 @@
     <origin
       xyz="-0.00077967 -0.3134 0.026811"
-      rpy="-3.1416 -1.5708 0" />
-    <axis
-      xyz="1 0 0" />
+      rpy="0 0 0" />
   </xacro:dc_motor>
   <xacro:dc_motor motor_name="osl_knee" robot_ns="/oslsim" parent_link="socket" child_link="osl_shank">
@@ -20,6 +18,4 @@
       xyz="-0.0073766 -0.062441 -0.4427"
       rpy="1.5708 0 0" />
-    <axis
-      xyz="0 0 1" />
   </xacro:dc_motor>
   <gazebo>
@@ -418,5 +414,5 @@
     <collision>
       <origin
-        xyz="0.029606 -0.065 0.05"
+        xyz="0.029606 -0.065 0.06"
         rpy="0 0 0" />
       <geometry>
@@ -454,6 +450,6 @@
     <inertial>
       <origin
-        xyz="0.029606 0.056108 0.013102"
-        rpy="0.175 0 0" />
+        xyz="0.029606 -0.056108 0.033102"
+        rpy="0.175 -1.5708 0" />
       <mass
         value="0.15826" />
@@ -469,5 +465,5 @@
       <origin
         xyz="0 0 0"
-        rpy="0.175 0 0" />
+        rpy="0.175 -1.5708 -3.1416" />
       <geometry>
         <mesh
@@ -482,6 +478,6 @@
     <collision>
       <origin
-        xyz="0.029606 0.065 0.05"
-        rpy="0 0 0" />
+        xyz="0.03 -0.065 0.03"
+        rpy="0 -1.5708 0" />
       <geometry>
         <box size="0.0675 0.025 0.2"/>
@@ -627,5 +623,5 @@
       <parent link="osl_foot"/>
       <child link="osl_foot_loadcell_link"/>
-      <origin xyz="0.03 0.065 0" rpy="0 0 0"/>
+      <origin xyz="-0.03 -0.065 0.03" rpy="0 0 0"/>
   </joint>
   <gazebo reference="osl_foot_loadcell_link">

Commit message: Added PID tuner.

File: urdf/oslsim.xacro (robot description, xacro)
@@ -59,5 +59,5 @@
       <axis xyz="1 0 0" />
       <limit effort="1" lower="-10.0" upper="100.0" velocity="1" />
-      <dynamics damping="0.2" friction="0.1"/>
+      <dynamics damping="0.05" friction="0.1"/>
   </joint>
   <link name="entity">
@@ -90,5 +90,5 @@
         rpy="0 0 0" />
       <mass
-        value="1.0" />
+        value="0.1" />
       <inertia
         ixx="0.001"
@@ -112,5 +112,5 @@
         rpy="1.5708 0 0" />
       <mass
-        value="5.5797" />
+        value="0.55797" />
       <inertia
         ixx="0.0451"
@@ -156,5 +156,5 @@
         rpy="1.5708 0 0" />
       <mass
-        value="5.5993" />
+        value="0.55993" />
       <inertia
         ixx="0.045555"
@@ -236,5 +236,5 @@
         rpy="0 0 0" />
       <mass
-        value="0.53649" />
+        value="0.1" />
       <inertia
         ixx="0.00092445"
@@ -280,5 +280,5 @@
         rpy="0 0 0" />
       <mass
-        value="0.5365" />
+        value="0.1" />
       <inertia
         ixx="0.00092446"
@@ -389,5 +389,5 @@
         rpy="-0.175 0 0" />
       <mass
-        value="0.15826" />
+        value="0.01" />
       <inertia
         ixx="0.00051563"
@@ -414,5 +414,5 @@
     <collision>
       <origin
-        xyz="0.029606 -0.065 0.06"
+        xyz="0.029606 -0.065 0.05"
         rpy="0 0 0" />
       <geometry>
@@ -453,5 +453,5 @@
         rpy="0.175 -1.5708 0" />
       <mass
-        value="0.15826" />
+        value="0.01" />
       <inertia
         ixx="0.00051564"
@@ -553,28 +553,4 @@
     </actuator>
   </transmission>
-  <!-- <joint name="osl_ankle"
-    type="revolute">
-    <origin
-      xyz="-0.00077967 -0.3134 0.026811"
-      rpy="-3.1416 -1.5708 0" />
-    <parent
-      link="osl_shank" />
-    <child
-      link="osl_foot" />
-    <axis
-      xyz="1 0 0" />
-    <dynamics damping="0.5" friction="0.5"/>
-    <limit effort="1.0" velocity="100" lower="-1.57" upper="1.57" />
-  </joint>
-  <transmission name="osl_ankle_transmission">
-    <type>transmission_interface/SimpleTransmission</type>
-    <joint name="osl_ankle">
-      <hardwareInterface>hardware_interface/EffortJointInterface</hardwareInterface>
-    </joint>
-    <actuator name="osl_ankle_motor">
-      <hardwareInterface>hardware_interface/EffortJointInterface</hardwareInterface>
-      <mechanicalReduction>1</mechanicalReduction>
-    </actuator>
-  </transmission> -->
   <link name="foot_heel">
     <inertial>
